File: HAVOC_PCB_4.0/HAVOC_Practice.kicad_sch (KiCad schematic)
At the start: 44 parts, among them J1 132134, J10 BATT/switch, J3 NG, J7 solenoid, J8 Micro_SD_Card, J9 BNO, Q1 NMOS, Q2 NMOS, Q3 NMOS, Q4 NMOS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

Commit message: six seven
Other:
- note added: "six seven"
Changed lines of the file:
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@@
+		)
+	)
+	(text "six seven"
+		(exclude_from_sim no)
+		(at 101.854 174.244 0)
+		(effects
+			(font
+				(size 1.27 1.27)
+			)
 		)
 	)

Commit message: added backup battery and fixed missing PWM lines
Parts:
- removed AE1: Antenna_Shield, SHC:antennaufl, symbol Device:Antenna_Shield
- added BT1: Battery_Cell, SHC:GPS_BATT, symbol Device:Battery_Cell
- added C4: 1.0uF, Capacitor_SMD:C_0603_1608Metric_Pad1.08x0.95mm_HandSolder, symbol Device:C
- added R7: 1K, Resistor_SMD:R_0603_1608Metric_Pad0.98x0.95mm_HandSolder, symbol Device:R
Connections:
- net +3V3: now also R7.1
- net GND: now also BT1.2 (-), C4.2
- net PWM1: now also U1.37 (CS3); no longer U1.14 (A0)
- net PWM2: now also U1.36 (CS2); no longer U1.15 (A1)
- net GPS_BATT: now reaches U9.22 (V_BCKP)
- net GPS_BATT: now also BT1.1 (+), C4.1, R7.2
- net at J10.1 (Pin_1): now also J10.2 (Pin_2); no longer D1.2 (A)
- net at J10.3 (Pin_3): now also D1.2 (A); no longer J10.2 (Pin_2)
- no-connect marks 49 -> 48
Other:
- moved on the sheet: 3V3reg1, C1, C2, C3, D1, R15, U3, U4
